Commit message: Ejemplo completo usando amcl

File: diff_drive_robot_description/urdf/diff_drive_robot.xacro (robot description, xacro)
@@ -3,6 +3,6 @@
 <xacro:include filename="$(find diff_drive_robot_description)/urdf/material.xacro"/>
 <xacro:include filename="$(find diff_drive_robot_description)/urdf/macro.xacro"/>
-<!-- Dummy -->
-<link name="dummy_link"/>
+<!-- Footprint -->
+<link name="robot_footprint"/>
 <!-- Chassis -->
 <link name="base_link">
@@ -33,6 +33,6 @@
   </visual>
 </gazebo>
-<joint name="dummy_joint" type="fixed">
-  <parent link="dummy_link"/>
+<joint name="robot_footprint_base_joint" type="fixed">
+  <parent link="robot_footprint"/>
   <child link="base_link"/>
 </joint>
@@ -140,5 +140,5 @@
 </gazebo>
 <joint name="base_left_wheel_joint" type="continuous">
-  <origin xyz="0 -0.125 0" rpy="${pi/2} 0 0"/>
+  <origin xyz="0 0.125 0" rpy="0 ${pi/2} ${pi/2}"/>
   <parent link="base_link"/>
   <child link="left_wheel_link"/>
@@ -176,5 +176,5 @@
 </gazebo>
 <joint name="base_right_wheel_joint" type="continuous">
-  <origin xyz="0 0.125 0" rpy="${pi/2} 0 0"/>
+  <origin xyz="0 -0.125 0" rpy="0 ${pi/2} ${pi/2}"/>
   <parent link="base_link"/>
   <child link="right_wheel_link"/>
@@ -212,5 +212,5 @@
 </gazebo>
 <joint name="laser_link" type="fixed">
-  <origin xyz="-0.15 0 0.085" rpy="0 0 0"/>
+  <origin xyz="0.15 0 0.085" rpy="0 0 0"/>
   <parent link="base_link"/>
   <child link="laser_link"/>

File: diff_drive_robot_gazebo/urdf/gazebo.xacro (robot description, xacro)
@@ -16,5 +16,5 @@
     <odometryTopic>diff_drive_robot/odom</odometryTopic>
     <odometryFrame>odom</odometryFrame>
-    <robotBaseFrame>base_link</robotBaseFrame>
+    <robotBaseFrame>robot_footprint</robotBaseFrame>
     <rosDebugLevel>0</rosDebugLevel>
     <publishWheelTF>false</publishWheelTF>
